File: Hardware/smartwatch-top.brd (EAGLE design)
At the start: 38 x 38 mm, 51 parts, among them U1 NRF52832_MODULE_MDBT42, U4 PCF8523

Commit message: features list
Parts:
- removed C1, C8: 1u, LinnesLab-Passives:C0603
- removed C13: 100n, LinnesLab-Passives:C0603
- removed C3: (no value), LinnesLab-Passives:C0603
- removed CORTEX2: CORTEX_DEBUG_PTH, LinnesLab-Connectors:2X5-PTH-1.27MM
- removed D2: (no value), LinnesLab-DiscreteSemi:USC
- removed L1: 10u, LinnesLab-Passives:L0603
- removed LED1: RED, LinnesLab-LED:LED-0603
- removed LED2: BLUE, LinnesLab-LED:LED-0603
- removed R6, R8, R9: 10k, LinnesLab-Passives:R0603
- removed SW1, SW2: (no value), LinnesLab-Switches:BUTTON-GULLWING
- removed U1: NRF52832_MODULE_MDBT42, LinnesLab-Microcontrollers:BLE_MODULE_RAYTAC_MDBT42
- removed U4: PCF8523, LinnesLab-Clocks:SO8
- removed XTAL1: 32.768kHz, LinnesLab-Clocks:2-SMD.NOLEAD.2.0MMTO1.2MM
- removed XTAL3: (no value), LinnesLab-Clocks:2-SMD.NOLEAD.2.0MMTO1.2MM
- added C26: 1u, LinnesLab-Passives:C0603
- added C27, C28: (no value), LinnesLab-Passives:C0603
- added C29, C30: 300p, LinnesLab-Passives:C0603
- added C31: 10u, LinnesLab-Passives:C0805
- added C32: 100n, LinnesLab-Passives:C0603
- added CORTEX3: CORTEX_DEBUG_PTH, LinnesLab-Connectors:2X5-PTH-1.27MM
- added D3: (no value), LinnesLab-DiscreteSemi:USC
- added JP2: (no value), LinnesLab-Switches:SMT-JUMPER_2_NO_SILK
- added L3: 10u, LinnesLab-Passives:L0603
- added LED3, LED5: RED, LinnesLab-LED:LED-0603
- added LED4: YELLOW, LinnesLab-LED:LED-0603
- added LED6: BLUE, LinnesLab-LED:LED-0603
- added R10, R19: 27, LinnesLab-Passives:R0603
- added R16, R17, R20, R21: 1k, LinnesLab-Passives:R0603
- added R18, R3, R4: 10k, LinnesLab-Passives:R0603
- added SW5, SW6: (no value), LinnesLab-Switches:BUTTON-GULLWING
- added U2: FT231XS, LinnesLab-DigitalIC:SSOP20_L
- added U5: NRF52832_MODULE_MDBT42, LinnesLab-Microcontrollers:BLE_MODULE_RAYTAC_MDBT42
- added U6: PCF8523, LinnesLab-Clocks:SO8
- added XTAL2: 32.7680kHz, LinnesLab-Clocks:2-SMD.NOLEAD.2.0MMTO1.2MM
- added XTAL4: 32.768kHz, LinnesLab-Clocks:2-SMD.NOLEAD.2.0MMTO1.2MM
- C2: value (none) -> 1u
- C4: value 300p -> 100n
- C5: value 300p -> 47p
- C6: value 10u -> 47p; device LinnesLab-Passives:C0805 -> LinnesLab-Passives:C0603
- R1, R2: value 1k -> 0
- moved C2 65.7 mm to (10.8, -6.05), turned to 180 degrees
- moved R2 62.9 mm to (-17.2, -5.38)
- moved R1 62.6 mm to (-17.2, -2.69)
- moved C6 51.9 mm to (77.0, 42.1)
- moved C5 41.7 mm to (77.0, 47.1)
- moved C4 38.2 mm to (77.0, 52.2)
- moved C19 15.2 mm to (7.57, 25.3)
- moved C14 15.2 mm to (4.83, 25.2)
- moved C15 15.2 mm to (6.22, 25.4)
- moved C17 15.2 mm to (8.89, 25.3)
- moved R13 7.55 mm to (6.20, 6.27)
- moved LDO2 4.76 mm to (13.3, 10.9)
- moved R5 4.67 mm to (11.4, 6.65), turned to 90 degrees
- moved C20 3.09 mm to (6.22, 2.62)
- moved C11 1.60 mm to (8.56, 6.38)
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Connections:
- removed net A0/0.02: U1.15
- removed net A1/0.03: U1.16
- removed net A2/0.04: U1.17
- removed net A3/0.05: U1.18
- removed net A4/0.28: U1.5
- removed net A5/0.29: U1.6
- removed net A6/P0.30: U1.7
- removed net A7/P0.31: U1.8
- removed net N$1: C2.2, U1.13, XTAL1.P$1
- removed net N$13: CORTEX2.8
- removed net N$19: U4.2, XTAL3.P$1
- removed net N$20: U4.1, XTAL3.P$2
- removed net P0.07: U1.20
- removed net P0.11: U1.25
- removed net P0.15: U1.29
- removed net P0.16: U1.30
- removed net P0.27: U1.4
- removed net RXD: U1.21
- removed net TXD: U1.19
- new net !CTS: JP2.2, U2.9
- new net FT3V3: U2.13
- new net N$18: LED3.C, R20.2
- new net N$21: LED4.C, R21.2
- new net N$22: U6.1, XTAL2.P$2
- new net N$27: C27.2, U5.13, XTAL4.P$1
- new net N$28: C28.1, U5.14, XTAL4.P$2
- new net N$29: LED5.A, R16.1
- new net N$30: LED6.A, R17.1
- new net N$31: L3.1, U5.10
- new net N$32: C26.1, L3.2, U5.9
- new net N$33: CORTEX3.8
- new net RXD.FT: U2.4
- new net RXD.NRF: R1.2, U5.21
- new net RXLED: R20.1, U2.17
- new net TXD.FT: R1.1, U2.20
- new net TXD.NRF: R2.2, U5.19
- new net TXLED: R21.1, U2.10
- net 3.3V: now also C2.1, C31.2, C4.2, CORTEX3.1, D3.-, LED3.A, LED4.A, R18.2, R3.2, R4.2, U2.14, U2.3, U5.11, U6.8; no longer C6.2, C8.1, CORTEX2.1, D2.-, R6.2, R8.2, R9.2, U1.11, U4.8
- net DFU: now also SW5.3, U5.34; no longer SW1.3, U1.34
- net DTR: now also C32.1, U2.1; no longer C13.1
- net FRST: now also U5.38; no longer U1.38
- net GND: now also C2.2, C26.2, C27.1, C28.2, C29.2, C30.2, C31.1, C4.1, CORTEX3.3, CORTEX3.5, CORTEX3.7, CORTEX3.9, JP2.1, LED5.C, LED6.C, SW5.1, SW6.3, U2.16, U2.6, U5.1, U5.12, U5.24, U5.39, U6.4; no longer C1.2, C2.1, C3.2, C4.2, C8.2, CORTEX2.3, CORTEX2.5, CORTEX2.7, CORTEX2.9, LED1.C, LED2.C, SW1.1, SW2.3, U1.1, U1.12, U1.24, U1.39, U4.4
- net LED1: now also R16.2, U5.31; no longer R1.2, U1.31
- net LED2: now also R17.2, U5.33; no longer R2.2, U1.33
- net MISO: now also U5.28; no longer U1.28
- net MOSI: now also U5.27; no longer U1.27
- net N$2: now also R2.1; no longer C3.1, U1.14, XTAL1.P$2
- net N$3: now also R4.1; no longer L1.1, U1.10
- net N$5: now also U6.2, XTAL2.P$1; no longer LED1.A, R1.1
- net N$7: now also R10.2, U2.12; no longer LED2.A, R2.1
- net N$8: now also R19.2, U2.11; no longer C1.1, L1.2, U1.9
- net P0.09/NFC1: now also C30.1, U5.22; no longer C5.1, U1.22
- net P0.10/NFC2: now also C29.1, U5.23; no longer C4.1, U1.23
- net RESET: now also C32.2, CORTEX3.10, D3.+, R18.1, SW6.1, U5.35; no longer C13.2, CORTEX2.10, D2.+, R6.1, SW2.1, U1.35
- net SCK: now also U5.26; no longer U1.26
- net SCL: now also U5.3, U6.6; no longer R8.1, U1.3, U4.6
- net SDA: now also R3.1, U5.2, U6.5; no longer R9.1, U1.2, U4.5
- net SWCLK: now also CORTEX3.4, U5.36; no longer CORTEX2.4, U1.36
- net SWDIO: now also CORTEX3.2, U5.37; no longer CORTEX2.2, U1.37
- net SWO: now also CORTEX3.6, U5.32; no longer CORTEX2.6, U1.32
- net USB+: now also C5.1, R19.1
- net USB-: now also C6.2, R10.1
- net VBAT: now also U6.3; no longer U4.3
- net V_USB: now also U2.15
