File: Hardware/smartwatch-top.sch (EAGLE design)
At the start: 51 parts, among them U1 NRF52832_MODULE_MDBT42, U4 PCF8523

Commit message: features list
Parts:
- removed C1, C8: 1u, LinnesLab-Passives:CAPACITOR0603
- removed C13: 100n, LinnesLab-Passives:CAPACITOR0603
- removed C3: (no value), LinnesLab-Passives:CAPACITOR0603
- removed CORTEX2: CORTEX_DEBUG_PTH, LinnesLab-Connectors:CORTEX_DEBUG_PTH
- removed D2: (no value), LinnesLab-DiscreteSemi:SCHOTTKY-USC
- removed L1: 10u, LinnesLab-Passives:INDUCTOR0603
- removed LED1: RED, LinnesLab-LED:LED0603
- removed LED2: BLUE, LinnesLab-LED:LED0603
- removed R6, R8, R9: 10k, LinnesLab-Passives:RESISTOR0603
- removed SW1, SW2: (no value), LinnesLab-Switches:SPST-PTS830GG140-COPY.1-3
- removed U1: NRF52832_MODULE_MDBT42, LinnesLab-Microcontrollers:NRF52832_MODULE_MDBT42
- removed U4: PCF8523, LinnesLab-Clocks:PCF8523
- removed XTAL1: 32.768kHz, LinnesLab-Clocks:CRYSTALECS-.327-12.5-12-C-TR
- removed XTAL3: (no value), LinnesLab-Clocks:CRYSTALECS-.327-12.5-12-C-TR
- added C26: 1u, LinnesLab-Passives:CAPACITOR0603
- added C27, C28: (no value), LinnesLab-Passives:CAPACITOR0603
- added C29, C30: 300p, LinnesLab-Passives:CAPACITOR0603
- added C31: 10u, LinnesLab-Passives:CAPACITOR0805
- added C32: 100n, LinnesLab-Passives:CAPACITOR0603
- added CORTEX3: CORTEX_DEBUG_PTH, LinnesLab-Connectors:CORTEX_DEBUG_PTH
- added D3: (no value), LinnesLab-DiscreteSemi:SCHOTTKY-USC
- added JP2: (no value), LinnesLab-Switches:JUMPER-SMT_2_NO_SILK
- added L3: 10u, LinnesLab-Passives:INDUCTOR0603
- added LED3, LED5: RED, LinnesLab-LED:LED0603
- added LED4: YELLOW, LinnesLab-LED:LED0603
- added LED6: BLUE, LinnesLab-LED:LED0603
- added R10, R19: 27, LinnesLab-Passives:RESISTOR0603
- added R16, R17, R20, R21: 1k, LinnesLab-Passives:RESISTOR0603
- added R18, R3, R4: 10k, LinnesLab-Passives:RESISTOR0603
- added SW5, SW6: (no value), LinnesLab-Switches:SPST-PTS830GG140-COPY.1-3
- added U2: FT231XS, LinnesLab-DigitalIC:FT231XS
- added U5: NRF52832_MODULE_MDBT42, LinnesLab-Microcontrollers:NRF52832_MODULE_MDBT42
- added U6: PCF8523, LinnesLab-Clocks:PCF8523
- added XTAL2: 32.7680kHz, LinnesLab-Clocks:CRYSTALECS-.327-12.5-12-C-TR
- added XTAL4: 32.768kHz, LinnesLab-Clocks:CRYSTALECS-.327-12.5-12-C-TR
- C2: value (none) -> 1u
- C4: value 300p -> 100n
- C5: value 300p -> 47p
- C6: value 10u -> 47p; device LinnesLab-Passives:CAPACITOR0805 -> LinnesLab-Passives:CAPACITOR0603
- R1, R2: value 1k -> 0
Connections:
- removed net A0/0.02: U1.P0.02/AIN0
- removed net A1/0.03: U1.P0.03/AIN1
- removed net A2/0.04: U1.P0.04/AIN2
- removed net A3/0.05: U1.P0.05/AIN3
- removed net A4/0.28: U1.P0.28/AIN4
- removed net A5/0.29: U1.P0.29/AIN5
- removed net A6/P0.30: U1.P0.30/AIN6
- removed net A7/P0.31: U1.P0.31/AIN7
- removed net N$1: C2.2, U1.P0.00/XL1, XTAL1.1
- removed net N$13: CORTEX2.NC/TDI
- removed net N$19: U4.OSCO, XTAL3.1
- removed net N$20: U4.OSCI, XTAL3.2
- removed net P0.07: U1.P0.07
- removed net P0.11: U1.P0.11
- removed net P0.15: U1.P0.15
- removed net P0.16: U1.P0.16
- removed net P0.27: U1.P0.27
- removed net RXD: U1.P0.08
- removed net TXD: U1.P0.06
- new net !CTS: JP2.2, U2.!CTS
- new net FT3V3: U2.3V3OUT
- new net N$18: LED3.C, R20.2
- new net N$21: LED4.C, R21.2
- new net N$22: U6.OSCI, XTAL2.2
- new net N$27: C27.2, U5.P0.00/XL1, XTAL4.1
- new net N$28: C28.1, U5.P0.01/XL2, XTAL4.2
- new net N$29: LED5.A, R16.1
- new net N$30: LED6.A, R17.1
- new net N$31: L3.1, U5.DCC
- new net N$32: C26.1, L3.2, U5.DEC4
- new net N$33: CORTEX3.NC/TDI
- new net RXD.FT: U2.RXD
- new net RXD.NRF: R1.2, U5.P0.08
- new net RXLED: R20.1, U2.CBUS1
- new net TXD.FT: R1.1, U2.TXD
- new net TXD.NRF: R2.2, U5.P0.06
- new net TXLED: R21.1, U2.CBUS2
- net 3.3V: now also C2.1, C31.2, C4.2, CORTEX3.VCC, D3.C, LED3.A, LED4.A, R18.2, R3.2, R4.2, U2.!RESET, U2.VCCIO, U5.VDD, U6.VDD; no longer C6.2, C8.1, CORTEX2.VCC, D2.C, R6.2, R8.2, R9.2, U1.VDD, U4.VDD
- net DFU: now also SW5.B, U5.P0.20; no longer SW1.B, U1.P0.20
- net DTR: now also C32.1, U2.!DTR; no longer C13.1
- net FRST: now also U5.P0.22; no longer U1.P0.22
- net GND: now also C2.2, C26.2, C27.1, C28.2, C29.2, C30.2, C31.1, C4.1, CORTEX3.GND@3, CORTEX3.GND@5, CORTEX3.GNDDTCT, CORTEX3.KEY, JP2.1, LED5.C, LED6.C, SW5.A, SW6.B, U2.GND@16, U2.GND@6, U5.GND@1, U5.GND@2, U5.GND@3, U5.GND@4, U6.VSS; no longer C1.2, C2.1, C3.2, C4.2, C8.2, CORTEX2.GND@3, CORTEX2.GND@5, CORTEX2.GNDDTCT, CORTEX2.KEY, LED1.C, LED2.C, SW1.A, SW2.B, U1.GND@1, U1.GND@2, U1.GND@3, U1.GND@4, U4.VSS
- net LED1: now also R16.2, U5.P0.17; no longer R1.2, U1.P0.17
- net LED2: now also R17.2, U5.P0.19; no longer R2.2, U1.P0.19
- net MISO: now also U5.P0.14; no longer U1.P0.14
- net MOSI: now also U5.P0.13; no longer U1.P0.13
- net N$2: now also R2.1; no longer C3.1, U1.P0.01/XL2, XTAL1.2
- net N$3: now also R4.1; no longer L1.1, U1.DCC
- net N$5: now also U6.OSCO, XTAL2.1; no longer LED1.A, R1.1
- net N$7: now also R10.2, U2.USBDM; no longer LED2.A, R2.1
- net N$8: now also R19.2, U2.USBDP; no longer C1.1, L1.2, U1.DEC4
- net P0.09/NFC1: now also C30.1, U5.P0.09; no longer C5.1, U1.P0.09
- net P0.10/NFC2: now also C29.1, U5.P0.10; no longer C4.1, U1.P0.10
- net RESET: now also C32.2, CORTEX3.!RESET, D3.A, R18.1, SW6.A, U5.P0.21/RESET; no longer C13.2, CORTEX2.!RESET, D2.A, R6.1, SW2.A, U1.P0.21/RESET
- net SCK: now also U5.P0.12; no longer U1.P0.12
- net SCL: now also U5.P0.26, U6.SCL; no longer R8.1, U1.P0.26, U4.SCL
- net SDA: now also R3.1, U5.P0.25, U6.SDA; no longer R9.1, U1.P0.25, U4.SDA
- net SWCLK: now also CORTEX3.SWDCLK/TCK, U5.SWDCLK; no longer CORTEX2.SWDCLK/TCK, U1.SWDCLK
- net SWDIO: now also CORTEX3.SWDIO/TMS, U5.SWDIO; no longer CORTEX2.SWDIO/TMS, U1.SWDIO
- net SWO: now also CORTEX3.SWO/TDO, U5.P0.18/SWO; no longer CORTEX2.SWO/TDO, U1.P0.18/SWO
- net USB+: now also C5.1, R19.1
- net USB-: now also C6.2, R10.1
- net V_USB: now also U2.VCC
Other:
- note added: "Additional notes for advanced users only"
- note added: "FTDI Serial-to-USB Converter"
- note added: "I don't remember if CTS needs to be grounded or left floating so here's a jumper to ground so it can be configued either way dynamically."
- note added: "I2C Address = 0x68h"
- note added: "Microcontroller Reset Circuit"
- note added: "Notes"
- note added: "PIN_DFU / P0.20: If this pin is detected to be at GND level at startup, the board will enter a special serial bootloader mode and will not execute any user code, going straight into bootloader mode. If you wish to use this pin as a standard GPIO, make sure that it is pulled high with a pullup resistor so that your code will execute normally when the MCU starts up. FRST/P0.22: Setting this pin to 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"
- note added: "SPECIAL / PORT / PIN ON PACKAGE / GPIO(D_or_A) / Comments Factory Reset / P0.22 / pin38 / DO NOT USE FOR ANY GPIO SWDIO / none / pin37 / reserved-not available for general GPIO SWCLK / none / pin36 / reserved-not available for general GPIO RESET / P0.21 / pin35 / reserved-not available for general GPIO DFU / P0.20 / pin34 / reserved-not available for general GPIO LED2 / P0.19 / pin33 / reserved f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"
- note added: "SPECIAL / PORT / PIN ON PACKAGE / GPIO(D_or_A) / Comments SDA / P0.25 / pin2 / D25 SCL / P0.26 / pin3 / D26 none / P0.27 / pin4 / D27 none / P0.28 / pin5 / D28_or_A4 / (low drive, low frequency IO) none / P0.29 / pin6 / D29_or_A5 / (low drive, low frequency IO) none / P0.30 / pin7 / D30_or_A6 none / P0.31 / pin8 / D31_or_A7 / (used for battery level monitoring on Adafruit boards)"
- note added: "SPECIAL / PORT / PIN ON PACKAGE / GPIO(D_or_A) / Comments none / P0.02 / pin15 / D2_or_A0 none / P0.03 / pin16 / D3_or_A1 none / P0.04 / pin17 / D4_or_A2 none / P0.05 / pin18 / D5_or_A3 TXD / P0.06 / pin19 / D6 / but reserved for Serial communication and programming none / P0.07 / pin20 / D7 RXD / P0.08 / pin21 / D8 / but reserved for Serial communication and programming NFC1 / P0.09 / pin22 / D9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"
- note added: "Some pins are noted as reserved and not available for general GPIO (unless you are an adavanced user) I2C, SPI, and SWD pins can be repurposed if you know what you are doing For Milestones, avoid repurposing NFC pins. For P0.19 (LED2), Adafruit's Bluetooth Low Energy libraries use this pin to indicated successful pairing. The LED blinks when the device is doing some Bluetooth process and stays li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"
- note added: "TXD goes to RX on the other device RXD goes to TX on the other device"
- note removed: "RTC"
- note removed: "USB RESET (DTR)"
- moved on the sheet: C2, C4, C5, C6, R1, R2, U$1, U$2
