File: Hardware/Bottom/smartwatch-bottom.brd (EAGLE design)
At the start: 33 x 33 mm, 31 parts, among them U2 AD5242-SO16

Commit message: Finished Take003
Parts:
- removed OP1: (no value), LinnesLab-AnalogIC:SOT23-5
- removed U$2: AD5171, LinnesLab-DigitalIC:SOT-23-8
- removed U2: AD5242-SO16, LinnesLab-DigitalIC:SO16
- added AD5171: AD5171, LinnesLab-DigitalIC:SOT-23-8
- added AD5242: AD5242-SO16, LinnesLab-DigitalIC:SO16
- added C10: 100n, LinnesLab-Passives:C0603
- added J1: (no value), LinnesLab-Connectors:1X07_1.27MM
- added LOGO1: REVISION.A, LinnesLab-Logos:REV.A
- added LOGO2: OSHW-LOGOS, LinnesLab-Logos:OSHW-LOGO-S
- added TIA: (no value), LinnesLab-AnalogIC:SOT23-5
- moved R3 30.3 mm to (33.1, 4.98), turned to 270 degrees
- moved C9 28.7 mm to (33.2, 14.5), turned to 90 degrees
- moved C8 26.9 mm to (29.6, 4.42)
- moved R2 25.5 mm to (29.6, 6.31), turned to 180 degrees
- moved R1 24.6 mm to (33.1, 9.11), turned to 270 degrees
- moved C4 21.1 mm to (25.9, 9.13), turned to 90 degrees
- moved IMU1 20.3 mm to (6.27, 27.9), turned to 90 degrees
- moved R10 20.0 mm to (25.0, 20.4), turned to 90 degrees
- moved C5 19.8 mm to (22.9, 10.1), turned to 180 degrees
- moved C7 19.8 mm to (29.6, 8.12), turned to 180 degrees
- moved R12 19.4 mm to (23.8, 7.36), turned to 270 degrees
- moved R4 19.2 mm to (29.6, 9.95)
- moved C2 19.1 mm to (21.8, 7.34), turned to 270 degrees
- moved C11 16.2 mm to (6.70, 23.7), turned to 0 degrees
- moved C6 15.6 mm to (13.9, 20.6), turned to 90 degrees
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Connections:
- removed net LED: Q2.3
- removed net LED.CTRL: U$2.8
- removed net PPG: C5.2, OP2.1, U2.14
- removed net TIA: C3.2, C8.1, OP1.1, U2.3
- new net A6/TIA: AD5242.3, C3.2, C8.1, J1.6, TIA.1
- new net A7/PPG: AD5242.14, C5.2, J1.7, OP2.1
- new net D29/LED.CTRL: AD5171.8, J1.5
- net 3.3V: now also AD5171.2, AD5171.6, AD5242.5, AD5242.6, J1.4, TIA.5; no longer OP1.5, U$2.2, U$2.6, U2.5, U2.6
- net G.A1: now also AD5242.2; no longer U2.2
- net G.A2: now also AD5242.16; no longer U2.16
- net G.O1: now also AD5242.1; no longer U2.1
- net G.O2: now also AD5242.13; no longer U2.13
- net G.W2: now also AD5242.15; no longer U2.15
- net GND: now also AD5171.3, AD5242.10, AD5242.11, AD5242.12, AD5242.9, C10.1, J1.3, TIA.2, TIA.3; no longer OP1.2, OP1.3, U$2.3, U2.10, U2.11, U2.12, U2.9
- net LED.C: now also Q2.3
- net N$12: now also AD5171.1, AD5171.7; no longer U$2.1, U$2.7
- net PD.C: now also AD5242.4, TIA.4; no longer OP1.4, U2.4
- net SCL: now also AD5171.4, AD5242.7, J1.2; no longer U$2.4, U2.7
- net SDA: now also AD5171.5, AD5242.8, J1.1; no longer U$2.5, U2.8
- net VREF: now also C10.2
Routing:
- net A6/TIA: track 0.00 -> 68.2 mm, vias 0 -> 4
- net A7/PPG: track 0.00 -> 54.6 mm
- net VREF: track 0.00 -> 35.3 mm, vias 0 -> 3
- net SDA: track 0.00 -> 35.2 mm
- net SCL: track 0.00 -> 35.1 mm, vias 0 -> 2
- net GND: track 0.00 -> 27.2 mm, vias 0 -> 15
- net PD.C: track 0.00 -> 25.0 mm, vias 0 -> 2
- net N$6: track 0.00 -> 22.5 mm
- net N$12: track 0.00 -> 20.2 mm
- net D29/LED.CTRL: track 0.00 -> 16.9 mm, vias 0 -> 2
- net G.W2: track 0.00 -> 16.4 mm, vias 0 -> 2
- net N$1: track 0.00 -> 15.8 mm
- net N$2: track 0.00 -> 9.15 mm, vias 0 -> 2
- net N$4: track 0.00 -> 8.59 mm
- net N$5: track 0.00 -> 6.30 mm
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- added copper zone on layer 1, net 3.3V
- added copper zone on layer 16, net GND
