File: Hardware/Bottom/ShaqJr-BOTTOM.brd (EAGLE design)
At the start: 33 x 33 mm, 35 parts

Commit message: completed take 007, may need to review polygons- gnd and 3.3v
Parts:
- added C14, C15, C16: 1u, LinnesLab-Passives:C0603
- added C17, C18: 4.7u, LinnesLab-Passives:C0603
- added CHRG1: MCP73831, LinnesLab-Power:SOT23-5
- added LDO1: MIC5504, LinnesLab-Power:SOT23-5
- added R13: (no value), LinnesLab-Passives:R0603
- added R14, R15, R16, R17: 100k, LinnesLab-Passives:R0603
- added U1: PCF8523, LinnesLab-Clocks:SO8
- added Y1: 32.7680kHz, LinnesLab-Clocks:2-SMD.NOLEAD.2.0MMTO1.2MM
Connections:
- new net A4/BATT: R15.1, R16.2
- new net D27/CHRG.STATUS: CHRG1.1, R14.1
- new net N$10: U1.1, Y1.P$2
- new net N$17: CHRG1.5, R13.2
- new net N$9: U1.2, Y1.P$1
- new net VBAT: U1.3
- new net VIN1: C15.2, C18.2, CHRG1.4, LDO1.1, LDO1.3, R14.2
- new net VLIPO: C17.1, CHRG1.3, R15.2
- net 3.3V: now also C14.1, C16.1, LDO1.5, R17.2, U1.8
- net GND: now also C14.2, C15.1, C16.2, C17.2, C18.1, CHRG1.2, LDO1.2, R13.1, R16.1, R17.1, U1.4
- net SCL: now also U1.6
- net SDA: now also U1.5

Commit message: Finished Take 008
Parts:
- removed C15, C16: 1u, LinnesLab-Passives:C0603
- removed C17, C18: 4.7u, LinnesLab-Passives:C0603
- removed CHRG1: MCP73831, LinnesLab-Power:SOT23-5
- removed LDO1: MIC5504, LinnesLab-Power:SOT23-5
- removed R13: (no value), LinnesLab-Passives:R0603
- removed R14, R15, R16, R17: 100k, LinnesLab-Passives:R0603
- moved C14 67.2 mm to (33.2, 32.6), turned to 270 degrees
- moved Y1 65.7 mm to (24.5, 32.7), turned to 90 degrees
- moved U1 61.6 mm to (28.8, 31.5)
- moved LOGO2 8.34 mm to (26.2, 27.2)
- moved C10 3.46 mm to (31.2, 25.6), turned to 180 degrees
- moved IMU1 0.37 mm to (6.27, 27.5)
- moved R9 0.36 mm to (19.0, 29.3)
- moved C13 0.17 mm to (5.25, 8.62)
- moved Q2 0.10 mm to (19.0, 26.8)
Connections:
- net A6/TIA renamed A5/TIA
- net A7/PPG renamed A4/PPG
- net D29/LED.CTRL renamed D30/LED.CTRL
- removed net A4/BATT: R15.1, R16.2
- removed net D27/CHRG.STATUS: CHRG1.1, R14.1
- removed net N$17: CHRG1.5, R13.2
- removed net VIN1: C15.2, C18.2, CHRG1.4, LDO1.1, LDO1.3, R14.2
- removed net VLIPO: C17.1, CHRG1.3, R15.2
- net 3.3V: no longer C16.1, LDO1.5, R17.2
- net GND: no longer C15.1, C16.2, C17.2, C18.1, CHRG1.2, LDO1.2, R13.1, R16.1, R17.1
Routing:
- net SDA: track 35.2 -> 62.4 mm, vias 0 -> 2
- net SCL: track 35.1 -> 60.9 mm, vias 2 -> 4
- net A5/TIA: track 68.2 -> 64.6 mm
- net GND: track 27.2 -> 29.5 mm, vias 15 -> 17
- net A4/PPG: track 54.6 -> 52.6 mm
- net N$9: track 0.00 -> 1.79 mm
- net N$10: track 0.00 -> 1.66 mm
