File: Hardware/Top/smartwatch-top.brd (EAGLE design)
At the start: 38 x 38 mm, 64 parts, among them U2 FT231XS, U5 NRF52832_MODULE_MDBT42, U6 PCF8523

Commit message: Finished Take003
Parts:
- removed C26: 1u, LinnesLab-Passives:C0603
- removed C27: (no value), LinnesLab-Passives:C0603
- removed C31: 10u, LinnesLab-Passives:C0805
- removed C32: 100n, LinnesLab-Passives:C0603
- removed CHRG2: MCP73831, LinnesLab-Power:SOT23-5
- removed D4, D5: (no value), LinnesLab-DiscreteSemi:USC
- removed LDO2: MIC5504, LinnesLab-Power:SOT23-5
- removed R19: 27, LinnesLab-Passives:R0603
- removed R20, R21: 1k, LinnesLab-Passives:R0603
- removed U5: NRF52832_MODULE_MDBT42, LinnesLab-Microcontrollers:BLE_MODULE_RAYTAC_MDBT42
- removed U6: PCF8523, LinnesLab-Clocks:SO8
- removed XTAL2: 32.7680kHz, LinnesLab-Clocks:2-SMD.NOLEAD.2.0MMTO1.2MM
- added C1, C8: 4.7u, LinnesLab-Passives:C0603
- added C13: 47p, LinnesLab-Passives:C0603
- added C3: 1u, LinnesLab-Passives:C0603
- added CHRG1: MCP73831, LinnesLab-Power:SOT23-5
- added D1, D2: (no value), LinnesLab-DiscreteSemi:USC
- added J1: (no value), LinnesLab-Connectors:1X02
- added LDO1: MIC5504, LinnesLab-Power:SOT23-5
- added R6: 100k, LinnesLab-Passives:R0603
- added R8, R9: 1k, LinnesLab-Passives:R0603
- added U1: NRF52832_MODULE_MDBT42, LinnesLab-Microcontrollers:BLE_MODULE_RAYTAC_MDBT42
- added U4: (no value), LinnesLab-Displays:UG-2864HSWEG01_0.96IN_NO-WRAPAROUND
- added Y2: 32.7680kHz, LinnesLab-Clocks:2-SMD.NOLEAD.2.0MMTO1.2MM
- C11: value 1u -> 100n
- C12: value 1u -> 47p
- C14: value 2.2uF -> 10uF; device LinnesLab-Passives:C0402 -> LinnesLab-Passives:C0603
- C15: value 2.2uF -> 100n; device LinnesLab-Passives:C0402 -> LinnesLab-Passives:C0603
- C16: value 10uF -> 2.2uF; device LinnesLab-Passives:C0603 -> LinnesLab-Passives:C0402
- C20: value 4.7u -> 2.2uF; device LinnesLab-Passives:C0603 -> LinnesLab-Passives:C0402
- C21: value 4.7u -> 1u
- C4: value 100n -> 10u; device LinnesLab-Passives:C0603 -> LinnesLab-Passives:C0805
- C5: value 47p -> (none)
- C6: value 47p -> 1u
- J2: device LinnesLab-Connectors:1X02 -> LinnesLab-Connectors:1X07_1.27MM
- R1, R2: value 0 -> 10k
- R10: value 27 -> 10k
- R11: value (none) -> 10k
- R12, R13: value 100k -> 27
- R14: value 100k -> 390k
- R15: value 100k -> 1k
- R17: value 1k -> 0
- R18: value 10k -> 0
- R3, R5: value 10k -> 100k
- R4: value 10k -> (none)
- R7: value 390k -> 100k
- U2: value FT231XS -> PCF8523; device LinnesLab-DigitalIC:SSOP20_L -> LinnesLab-Clocks:SO8
- U3: value (none) -> FT231XS; device LinnesLab-Displays:UG-2864HSWEG01_0.96IN_NO-WRAPAROUND -> LinnesLab-DigitalIC:SSOP20_L
- moved C6 89.7 mm to (7.80, -15.0), turned to 270 degrees
- moved R15 80.5 mm to (80.8, 44.3), turned to 0 degrees
- moved C12 77.9 mm to (77.0, 42.1), turned to 0 degrees
- moved C15 75.7 mm to (77.0, 52.2), turned to 0 degrees
- moved R13 70.8 mm to (64.2, 46.8), turned to 0 degrees
- moved R12 67.3 mm to (63.5, 50.0), turned to 0 degrees
- moved C11 64.8 mm to (73.4, 5.79), turned to 270 degrees
- moved C4 53.3 mm to (46.5, 8.59)
- moved C5 52.4 mm to (49.4, 2.62)
- moved R18 52.4 mm to (53.7, 56.3), turned to 0 degrees
- moved U2 48.9 mm to (47.1, -12.6), turned to 0 degrees
- moved C21 46.6 mm to (48.9, -9.04), turned to 180 degrees
- moved R17 45.8 mm to (53.7, 59.0), turned to 0 degrees
- moved R10 44.3 mm to (68.4, 6.05), turned to 90 degrees
- moved U3 44.0 mm to (45.3, 54.8), turned to 270 degrees
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- renumbered C28 to C7, C29 to C10, C30 to C9, CORTEX3 to DEBUG1, JP2 to JP1, L3 to L1, LED5 to LED1, LED6 to LED2, SD2 to SD1, SW5 to SW1, SW6 to SW2, U$1 to SW3, U$2 to SW4, USB2 to USB1, XTAL4 to Y1
Connections:
- removed net BATT: R13.1, R14.2
- removed net CD1: SD1.CD1
- removed net CHRG.STAT: CHRG2.1, R12.1
- removed net CS.OLED: U3.13
- removed net DC.OLED: U3.15
- removed net N$3 (its old number): R4.1
- removed net RESET.OLED: U3.14
- removed net SD.CS: SD1.2
- removed net SW1: SW3.A1, SW4.A1
- new net A4/BATT: R6.1, R7.2, U1.5
- new net A6/TIA: J2.6, U1.7
- new net A7/PPG: J2.7, U1.8
- new net D11/SW1: SW3.A1, U1.25
- new net D15/SW2: SW4.A1, U1.29
- new net D16/CS.OLED: U1.30, U4.13
- new net D27/CHRG.STATUS: CHRG1.1, R3.1, U1.4
- new net D29/LED.CTRL: J2.5, U1.6
- new net D3/RESET.OLED: U1.16, U4.14
- new net D4/DC.OLED: U1.17, U4.15
- new net D5/CD1: SD1.CD1, U1.18
- new net D7/SD.CS: SD1.2, U1.20
- new net N$2: R18.1
- net !CTS: now also U3.9; no longer U2.9
- net 3.3V: now also C15.2, C20.2, C21.1, C6.1, J2.4, LDO1.5, R1.2, R10.2, R2.2, R5.2, U1.11, U2.8, U3.14, U3.3, U4.6, U4.9; no longer C12.1, C17.2, C2.1, C31.2, LDO2.5, R15.2, R18.2, R3.2, R4.2, U2.14, U2.3, U3.6, U3.9, U5.11, U6.8
- net DFU: now also U1.34; no longer U5.34
- net DTR: now also C11.1, U3.1; no longer C32.1, U2.1
- net FRST: now also U1.38; no longer U5.38
- net FT3V3: now also U3.13; no longer U2.13
- net GND: now also C1.1, C12.1, C13.2, C14.1, C15.1, C20.1, C21.2, C3.1, C5.1, C6.2, C8.2, CHRG1.2, J1.1, J2.3, LDO1.2, R14.2, R4.1, R7.1, U1.1, U1.12, U1.24, U1.39, U2.4, U3.16, U3.6, U4.1, U4.10, U4.12, U4.29, U4.30, U4.8; no longer C11.1, C12.2, C16.1, C18.1, C20.2, C21.1, C26.2, C27.1, C31.1, C5.2, C6.1, CHRG2.2, J2.1, LDO2.2, R14.1, R15.1, R7.2, U2.16, U2.6, U3.1, U3.10, U3.12, U3.29, U3.30, U3.8, U5.1, U5.12, U5.24, U5.39, U6.4
- net LED1: now also R8.2, U1.31; no longer R16.2, U5.31
- net LED2: now also R9.2, U1.33; no longer R17.2, U5.33
- net MISO: now also U1.28; no longer U5.28
- net MOSI: now also U1.27, U4.19; no longer U3.19, U5.27
- net N$10: now also C18.1, U4.3; no longer C14.1, U3.3
- net N$11: now also C16.2, U4.4; no longer C15.2, U3.4
- net N$12: now also C16.1, U4.5; no longer C15.1, U3.5
- net N$14: now also C14.2, U4.28; no longer C16.2, U3.28
- net N$15: now also C17.2, U4.27; no longer C18.2, U3.27
- net N$17: now also CHRG1.5, R4.2; no longer CHRG2.5, R11.2
- net N$18: now also R15.2; no longer R20.2
- net N$21: now also R16.2; no longer R21.2
- net N$22: now also U2.1, Y2.P$2; no longer U6.1, XTAL2.P$2
- net N$27: now also C5.2, U1.13; no longer C27.2, U5.13
- net N$28: now also U1.14; no longer U5.14
- net N$29: now also R8.1; no longer R16.1
- net N$30: now also R9.1; no longer R17.1
- net N$31: now also U1.10; no longer U5.10
- net N$32: now also C2.1, U1.9; no longer C26.1, U5.9
- net N$4: now also R11.2, U4.11; no longer R5.2, U3.11
- net N$5: now also U2.2, Y2.P$1; no longer U6.2, XTAL2.P$1
- net N$6: now also R14.1, U4.26; no longer R7.1, U3.26
- net N$7: now also R12.2, U3.12; no longer R10.2, U2.12
- net N$8: now also R13.2, U3.11; no longer R19.2, U2.11
- net N$9: now also C18.2, U4.2; no longer C14.2, U3.2
- net P0.09/NFC1: now also U1.22; no longer U5.22
- net P0.10/NFC2: now also U1.23; no longer U5.23
- net RESET: now also C11.2, R10.1, U1.35; no longer C32.2, R18.1, U5.35
- net RXD.FT: now also U3.4; no longer U2.4
- net RXD.NRF: now also R17.2, U1.21; no longer R1.2, U5.21
- net RXLED: now also R15.1, U3.17; no longer R20.1, U2.17
- net SCK: now also U1.26, U4.18; no longer U3.18, U5.26
- net SCL: now also J2.2, U1.3, U2.6; no longer U5.3, U6.6
- net SDA: now also J2.1, R1.1, U1.2, U2.5; no longer R3.1, U5.2, U6.5
- net SWCLK: now also U1.36; no longer U5.36
- net SWDIO: now also U1.37; no longer U5.37
- net SWO: now also U1.32; no longer U5.32
- net TXD.FT: now also R17.1, U3.20; no longer R1.1, U2.20
- net TXD.NRF: now also R18.2, U1.19; no longer R2.2, U5.19
- net TXLED: now also R16.1, U3.10; no longer R21.1, U2.10
- net USB+: now also C13.1, R13.1; no longer C5.1, R19.1
- net USB-: now also C12.2, R12.1; no longer C6.2, R10.1
- net VBAT: now also U2.3; no longer U6.3
- net VIN: now also C1.2, C3.2, CHRG1.4, D1.-, D2.-, LDO1.1, LDO1.3, R3.2; no longer C11.2, C21.2, CHRG2.4, D4.-, D5.-, LDO2.1, LDO2.3, R12.2
- net VLIPO: now also C8.1, CHRG1.3, D1.+, J1.2, R6.2; no longer C20.1, CHRG2.3, D4.+, J2.2, R13.2
- net V_USB: now also D2.+, U3.15; no longer D5.+, U2.15
