File: Hardware/Top/smartwatch-top.sch (EAGLE design)
At the start: 64 parts, among them U2 FT231XS, U5 NRF52832_MODULE_MDBT42, U6 PCF8523

Commit message: Finished Take003
Parts:
- removed C26: 1u, LinnesLab-Passives:CAPACITOR0603
- removed C27: (no value), LinnesLab-Passives:CAPACITOR0603
- removed C31: 10u, LinnesLab-Passives:CAPACITOR0805
- removed C32: 100n, LinnesLab-Passives:CAPACITOR0603
- removed R19: 27, LinnesLab-Passives:RESISTOR0603
- removed R20, R21: 1k, LinnesLab-Passives:RESISTOR0603
- removed U6: PCF8523, LinnesLab-Clocks:PCF8523
- added C1, C8: 4.7u, LinnesLab-Passives:CAPACITOR0603
- added C13: 47p, LinnesLab-Passives:CAPACITOR0603
- added C3: 1u, LinnesLab-Passives:CAPACITOR0603
- added J1: (no value), LinnesLab-Connectors:CONN_02
- added R6: 100k, LinnesLab-Passives:RESISTOR0603
- added R8, R9: 1k, LinnesLab-Passives:RESISTOR0603
- added U4: (no value), LinnesLab-Displays:DISP_OLED_UG-2864HSWEG01-NO-WRAPAROUND
- C11: value 1u -> 100n
- C12: value 1u -> 47p
- C14: value 2.2uF -> 10uF; device LinnesLab-Passives:CAPACITOR0402 -> LinnesLab-Passives:CAPACITOR0603
- C15: value 2.2uF -> 100n; device LinnesLab-Passives:CAPACITOR0402 -> LinnesLab-Passives:CAPACITOR0603
- C16: value 10uF -> 2.2uF; device LinnesLab-Passives:CAPACITOR0603 -> LinnesLab-Passives:CAPACITOR0402
- C20: value 4.7u -> 2.2uF; device LinnesLab-Passives:CAPACITOR0603 -> LinnesLab-Passives:CAPACITOR0402
- C21: value 4.7u -> 1u
- C4: value 100n -> 10u; device LinnesLab-Passives:CAPACITOR0603 -> LinnesLab-Passives:CAPACITOR0805
- C5: value 47p -> (none)
- C6: value 47p -> 1u
- J2: device LinnesLab-Connectors:CONN_02 -> LinnesLab-Connectors:CONN_07-1.27MM
- R1, R2: value 0 -> 10k
- R10: value 27 -> 10k
- R11: value (none) -> 10k
- R12, R13: value 100k -> 27
- R14: value 100k -> 390k
- R15: value 100k -> 1k
- R17: value 1k -> 0
- R18: value 10k -> 0
- R3, R5: value 10k -> 100k
- R4: value 10k -> (none)
- R7: value 390k -> 100k
- U2: value FT231XS -> PCF8523; device LinnesLab-DigitalIC:FT231XS -> LinnesLab-Clocks:PCF8523; DIGIKEY (none) -> 568-5306-1-ND; I2C_ADDRESS (none) -> 0x68h; MFN (none) -> PCF8523T/1,118; MFN_MANUFACTURER (none) -> NXP USA Inc.
- U3: value (none) -> FT231XS; device LinnesLab-Displays:DISP_OLED_UG-2864HSWEG01-NO-WRAPAROUND -> LinnesLab-DigitalIC:FT231XS
- renumbered C28 to C7, C29 to C10, C30 to C9, CHRG2 to CHRG1, CORTEX3 to DEBUG1, D4 to D1, D5 to D2, JP2 to JP1, L3 to L1, LDO2 to LDO1, LED5 to LED1, LED6 to LED2, SD2 to SD1, SW5 to SW1, SW6 to SW2, U$1 to SW3, U$2 to SW4, U5 to U1, USB2 to USB1, XTAL2 to Y2, XTAL4 to Y1
Connections:
- removed net BATT: R13.1, R14.2
- removed net CD1: SD1.CARD_DETECT
- removed net CHRG.STAT: CHRG1.STAT, R12.1
- removed net CS.OLED: U3./CS
- removed net DC.OLED: U3.DC/I2C_SA0
- removed net N$3 (its old number): R4.1
- removed net RESET.OLED: U3./RES
- removed net SD.CS: SD1.CS
- removed net SW1: SW3.1, SW4.1
- new net A4/BATT: R6.1, R7.2, U1.P0.28/AIN4
- new net A6/TIA: J2.6, U1.P0.30/AIN6
- new net A7/PPG: J2.7, U1.P0.31/AIN7
- new net D11/SW1: SW3.1, U1.P0.11
- new net D15/SW2: SW4.1, U1.P0.15
- new net D16/CS.OLED: U1.P0.16, U4./CS
- new net D27/CHRG.STATUS: CHRG1.STAT, R3.1, U1.P0.27
- new net D29/LED.CTRL: J2.5, U1.P0.29/AIN5
- new net D3/RESET.OLED: U1.P0.03/AIN1, U4./RES
- new net D4/DC.OLED: U1.P0.04/AIN2, U4.DC/I2C_SA0
- new net D5/CD1: SD1.CARD_DETECT, U1.P0.05/AIN3
- new net D7/SD.CS: SD1.CS, U1.P0.07
- new net N$2: R18.1
- net !CTS: now also U3.!CTS; no longer U2.!CTS
- net 3.3V: now also C15.2, C20.2, C21.1, C6.1, J2.4, R1.2, R10.2, R2.2, R5.2, U2.VDD, U3.!RESET, U3.VCCIO, U4.VBAT, U4.VDD; no longer C12.1, C17.2, C2.1, C31.2, R15.2, R18.2, R3.2, R4.2, U2.!RESET, U2.VCCIO, U3.VBAT, U3.VDD, U6.VDD
- net DTR: now also C11.1, U3.!DTR; no longer C32.1, U2.!DTR
- net FT3V3: now also U3.3V3OUT; no longer U2.3V3OUT
- net GND: now also C1.1, C12.1, C13.2, C14.1, C15.1, C20.1, C21.2, C3.1, C5.1, C6.2, C8.2, J1.1, J2.3, R14.2, R4.1, R7.1, U2.VSS, U3.GND@16, U3.GND@6, U4.BS0, U4.BS2, U4.NC(GND)@1, U4.NC(GND)@2, U4.VLSS, U4.VSS; no longer C11.1, C12.2, C16.1, C18.1, C20.2, C21.1, C26.2, C27.1, C31.1, C5.2, C6.1, J2.1, R14.1, R15.1, R7.2, U2.GND@16, U2.GND@6, U3.BS0, U3.BS2, U3.NC(GND)@1, U3.NC(GND)@2, U3.VLSS, U3.VSS, U6.VSS
- net LED1: now also R8.2; no longer R16.2
- net LED2: now also R9.2; no longer R17.2
- net MOSI: now also U4.D1/SPI_SDIN/I2C_SDA; no longer U3.D1/SPI_SDIN/I2C_SDA
- net N$10: now also C18.1, U4.C2N; no longer C14.1, U3.C2N
- net N$11: now also C16.2, U4.C1P; no longer C15.2, U3.C1P
- net N$12: now also C16.1, U4.C1N; no longer C15.1, U3.C1N
- net N$14: now also C14.2, U4.VCC; no longer C16.2, U3.VCC
- net N$15: now also C17.2, U4.VCOMH; no longer C18.2, U3.VCOMH
- net N$17: now also R4.2; no longer R11.2
- net N$18: now also R15.2; no longer R20.2
- net N$21: now also R16.2; no longer R21.2
- net N$22: now also U2.OSCI; no longer U6.OSCI
- net N$27: now also C5.2; no longer C27.2
- net N$29: now also R8.1; no longer R16.1
- net N$30: now also R9.1; no longer R17.1
- net N$32: now also C2.1; no longer C26.1
- net N$4: now also R11.2, U4.BS1; no longer R5.2, U3.BS1
- net N$5: now also U2.OSCO; no longer U6.OSCO
- net N$6: now also R14.1, U4.IREF; no longer R7.1, U3.IREF
- net N$7: now also R12.2, U3.USBDM; no longer R10.2, U2.USBDM
- net N$8: now also R13.2, U3.USBDP; no longer R19.2, U2.USBDP
- net N$9: now also C18.2, U4.C2P; no longer C14.2, U3.C2P
- net RESET: now also C11.2, R10.1; no longer C32.2, R18.1
- net RXD.FT: now also U3.RXD; no longer U2.RXD
- net RXD.NRF: now also R17.2; no longer R1.2
- net RXLED: now also R15.1, U3.CBUS1; no longer R20.1, U2.CBUS1
- net SCK: now also U4.D0/SPI_SCLK/I2C_SCK; no longer U3.D0/SPI_SCLK/I2C_SCK
- net SCL: now also J2.2, U2.SCL; no longer U6.SCL
- net SDA: now also J2.1, R1.1, U2.SDA; no longer R3.1, U6.SDA
- net TXD.FT: now also R17.1, U3.TXD; no longer R1.1, U2.TXD
- net TXD.NRF: now also R18.2; no longer R2.2
- net TXLED: now also R16.1, U3.CBUS2; no longer R21.1, U2.CBUS2
- net USB+: now also C13.1, R13.1; no longer C5.1, R19.1
- net USB-: now also C12.2, R12.1; no longer C6.2, R10.1
- net VIN: now also C1.2, C3.2, R3.2; no longer C11.2, C21.2, R12.2
- net VLIPO: now also C8.1, J1.2, R6.2; no longer C20.1, J2.2, R13.2
- net V_USB: now also U3.VCC; no longer U2.VCC
Other:
- note added: "Connection to bottom board"
- note added: "Digital Output"
- moved on the sheet: C11, C12, C14, C15, C16, C17, C18, C2, C20, C21, C4, C5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
