File: Hardware/Top/ShaqJr-TOP.sch (EAGLE design)
At the start: 65 parts, among them SW3 SWITCH.MOM, SW4 SWITCH.MOM, U1 NRF52832_MODULE_MDBT42, U2 PCF8523, U3 FT231XS, Y1 32.768kHz, Y2 32.7680kHz

Commit message: completed take 007, may need to review polygons- gnd and 3.3v
Parts:
- removed C10, C9: 300p, LinnesLab-Passives:CAPACITOR0603
- removed C21: 1u, LinnesLab-Passives:CAPACITOR0603
- removed SD1: (no value), LinnesLab-Connectors:MICROSD
- removed U2: PCF8523, LinnesLab-Clocks:PCF8523
- removed Y2: 32.7680kHz, LinnesLab-Clocks:CRYSTALECS-.327-12.5-12-C-TR
- added R19, R20: 100k, LinnesLab-Passives:RESISTOR0603
- C1: value 4.7u -> 1u
- C17: device LinnesLab-Passives:CAPACITOR0402 -> LinnesLab-Passives:CAPACITOR0603
- C6: value 1u -> 4.7u
- R3: value 100k -> (none)
- R4: value (none) -> 100k
Connections:
- removed net A6/TIA: J2.6, U1.P0.30/AIN6
- removed net A7/PPG: J2.7, U1.P0.31/AIN7
- removed net CD2: SD1.CARD_DETECT1
- removed net D29/LED.CTRL: J2.5, U1.P0.29/AIN5
- removed net N$2: R18.1
- removed net N$22: U2.OSCI, Y2.2
- removed net N$3: R2.1
- removed net N$5: U2.OSCO, Y2.1
- new net A4/PPG: J2.7, U1.P0.28/AIN4
- new net A5/TIA: J2.6, U1.P0.29/AIN5
- new net A7/BATT: R6.1, R7.2, U1.P0.31/AIN7
- new net D30/LED.CTRL: J2.5, U1.P0.30/AIN6
- net 3.3V: now also C3.1, R20.2; no longer C21.1, C6.1, R5.2, SD1.VDD, U2.VDD
- net A4/BATT: now also R19.2, R5.1; no longer R6.1, R7.2, U1.P0.28/AIN4
- net D27/CHRG.STATUS: now also R4.1; no longer R3.1
- net D5/CD1: no longer SD1.CARD_DETECT
- net D7/SD.CS: no longer SD1.CS
- net GND: now also C3.2, C8.1, R19.1, R20.1, R3.1; no longer C10.2, C21.2, C3.1, C8.2, C9.2, R4.1, R5.1, SD1.GND, SD1.GND1, SD1.VSS, U2.VSS
- net MISO: no longer SD1.DATA_OUT
- net MOSI: no longer SD1.DATA_IN
- net N$17: now also R3.2; no longer R4.2
- net P0.09/NFC1: no longer C9.1
- net P0.10/NFC2: no longer C10.1
- net RXD.FT: now also R18.1
- net SCK: no longer SD1.SCLK
- net SCL: now also R2.1; no longer U2.SCL
- net SDA: no longer U2.SDA
- net VIN: now also C8.2, R4.2; no longer C3.2, R3.2
- net VLIPO: now also C6.1, R5.2; no longer C8.1
Other:
- note removed: "Connect MISO, MOSI, and SCK to appropriate pins on microcontroller. Those are SPI pins and are generally prespecified. You have more flexibility with the SD.CS pin."
- note removed: "I2C Address = 0x68h"
- note removed: "Real-Time Clock"
- note removed: "SD Card"
- moved on the sheet: C1, C3, C6, C8, R3, R4, R5

Commit message: Finished Take 008
Parts:
- removed C19, C20: 2.2uF, LinnesLab-Passives:CAPACITOR0402
- removed R18: 0, LinnesLab-Passives:RESISTOR0603
- removed R19, R20: 100k, LinnesLab-Passives:RESISTOR0603
- removed SW2: (no value), LinnesLab-Switches:SPST-PTS830GG140-COPY.1-3
- removed U4: (no value), LinnesLab-Displays:DISP_OLED_UG-2864HSWEG01-NO-WRAPAROUND
- added C10: 47p, LinnesLab-Passives:CAPACITOR0603
- added C9: 100n, LinnesLab-Passives:CAPACITOR0603
- added RESET: (no value), LinnesLab-Switches:SPST-PTS830GG140-COPY.1-3
- added U2: FT231XS, LinnesLab-DigitalIC:FT231XS
- C1: value 1u -> 4.7u
- C11: value 100n -> 47p
- C12: value 47p -> 10uF
- C13: value 47p -> 100n
- C14: value 10uF -> 2.2uF; device LinnesLab-Passives:CAPACITOR0603 -> LinnesLab-Passives:CAPACITOR0402
- C15: value 100n -> 2.2uF
- C17: device LinnesLab-Passives:CAPACITOR0603 -> LinnesLab-Passives:CAPACITOR0402
- C6: value 4.7u -> 1u
- R11: value 10k -> 27
- R13: value 27 -> 390k
- R14: value 390k -> 1k
- R16: value 1k -> 0
- R3: value (none) -> 100k
- R4: value 100k -> 5k
- R7: value 100k -> 1k
- R9: value 1k -> 10k
- U3: value FT231XS -> (none); device LinnesLab-DigitalIC:FT231XS -> LinnesLab-Displays:DISP_OLED_UG-2864HSWEG01-NO-WRAPAROUND
Connections:
- removed net A4/BATT: R19.2, R5.1
- net !CTS: now also U2.!CTS; no longer U3.!CTS
- net 3.3V: now also C13.2, C17.2, C18.2, C6.1, R9.2, U2.!RESET, U2.VCCIO, U3.VBAT, U3.VDD; no longer C15.2, C19.2, C20.2, C3.1, R10.2, R20.2, U3.!RESET, U3.VCCIO, U4.VBAT, U4.VDD
- net A7/BATT: now also R5.1, R6.2; no longer R6.1, R7.2
- net D16/CS.OLED: now also U3./CS; no longer U4./CS
- net D27/CHRG.STATUS: now also R3.1; no longer R4.1
- net D3/RESET.OLED: now also U3./RES; no longer U4./RES
- net D4/DC.OLED: now also U3.DC/I2C_SA0; no longer U4.DC/I2C_SA0
- net DTR: now also C9.1, U2.!DTR; no longer C11.1, U3.!DTR
- net FT3V3: now also U2.3V3OUT; no longer U3.3V3OUT
- net GND: now also C10.1, C11.2, C13.1, C18.1, C3.1, C8.2, R10.1, R13.2, R4.1, R6.1, RESET.B, U2.GND@16, U2.GND@6, U3.BS0, U3.BS2, U3.NC(GND)@1, U3.NC(GND)@2, U3.VLSS, U3.VSS; no longer C13.2, C14.1, C19.1, C20.1, C3.2, C8.1, R11.1, R14.2, R19.1, R20.1, R3.1, R7.1, SW2.B, U3.GND@16, U3.GND@6, U4.BS0, U4.BS2, U4.NC(GND)@1, U4.NC(GND)@2, U4.VLSS, U4.VSS
- net LED1: now also R7.2; no longer R8.2
- net LED2: now also R8.2; no longer R9.2
- net MOSI: now also U3.D1/SPI_SDIN/I2C_SDA; no longer U4.D1/SPI_SDIN/I2C_SDA
- net N$10: now also C16.1, U3.C2N; no longer C18.1, U4.C2N
- net N$11: now also C14.2, U3.C1P; no longer C16.2, U4.C1P
- net N$12: now also C14.1, U3.C1N; no longer C16.1, U4.C1N
- net N$14: now also C12.2, U3.VCC; no longer C14.2, U4.VCC
- net N$15: now also C15.2, U3.VCOMH; no longer C17.2, U4.VCOMH
- net N$17: now also R4.2; no longer R3.2
- net N$18: now also R14.2; no longer R15.2
- net N$21: now also R15.2; no longer R16.2
- net N$29: now also R7.1; no longer R8.1
- net N$30: now also R8.1; no longer R9.1
- net N$4: now also R10.2, U3.BS1; no longer R11.2, U4.BS1
- net N$6: now also R13.1, U3.IREF; no longer R14.1, U4.IREF
- net N$7: now also R11.2, U2.USBDM; no longer R12.2, U3.USBDM
- net N$8: now also R12.2, U2.USBDP; no longer R13.2, U3.USBDP
- net N$9: now also C16.2, U3.C2P; no longer C18.2, U4.C2P
- net RESET: now also C9.2, R9.1, RESET.A; no longer C11.2, R10.1, SW2.A
- net RXD.FT: now also R17.1, U2.RXD; no longer R18.1, U3.RXD
- net RXD.NRF: now also R16.2; no longer R17.2
- net RXLED: now also R14.1, U2.CBUS1; no longer R15.1, U3.CBUS1
- net SCK: now also U3.D0/SPI_SCLK/I2C_SCK; no longer U4.D0/SPI_SCLK/I2C_SCK
- net TXD.FT: now also R16.1, U2.TXD; no longer R17.1, U3.TXD
- net TXD.NRF: now also R17.2; no longer R18.2
- net TXLED: now also R15.1, U2.CBUS2; no longer R16.1, U3.CBUS2
- net USB+: now also C11.1, R12.1; no longer C13.1, R13.1
- net USB-: now also C10.2, R11.1; no longer C12.2, R12.1
- net VIN: now also C3.2, R3.2; no longer C8.2, R4.2
- net VLIPO: now also C8.1; no longer C6.1, R6.2
- net V_USB: now also U2.VCC; no longer U3.VCC
Other:
- note added: "0 Ohm Resistors in case Orlando mixed up TX/RX"
- note added: "Diodes switch from LiPo power to USB when USB is connected The USB power then charges the battery"
- note added: "Headers connecting top and bottom boards"
- note added: "R3 sets charge current I_charge = 1000V/R3 per MCP73831 datasheet"
- note added: "Shaq Jr. Basic Top Revision A Date: Monday, July 16, 2020 Author: Akio"
- note added: "Voltage divider used to monitor battery voltage"
- moved on the sheet: C1, C11, C12, C13, C14, C15, C16, C17, C18, C3, C6, C8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
